File: 141 FC.kicad_pcb (KiCad board)
At the start: 2 copper layers, 45 parts, among them U2 TL431DBZ, U3 STM32H723ZGIx, Y1 ABM8G-24.000MHZ-4Y-T, Y2 ABS06-32.768KHZ-1-T

Commit message: Almost Complete Schematic
Parts:
- added C16: 100uF/6.3V, Capacitor_Tantalum_SMD:CP_EIA-3528-12_Kemet-T, F.Cu at (-66.5, 153.6)
- added C17: 100uF/6.3V, Capacitor_Tantalum_SMD:CP_EIA-3528-12_Kemet-T, F.Cu at (-66.5, 157.9)
- added C31: 4.7uF, Capacitor_SMD:C_0805_2012Metric, F.Cu at (-30.4, 167.9)
- added C32: 100nF, Capacitor_SMD:C_0805_2012Metric, F.Cu at (-30.4, 170.9)
- added C33: 100nF, Capacitor_SMD:C_0805_2012Metric, F.Cu at (-30.4, 173.9)
- added C34: 1uF, Capacitor_SMD:C_0805_2012Metric, F.Cu at (-56.7, 141.1)
- added C35: 100nF, Capacitor_SMD:C_0805_2012Metric, F.Cu at (-56.7, 144.1)
- added C36: 1uF, Capacitor_SMD:C_0805_2012Metric, F.Cu at (-56.7, 147.1)
- added C37: 100nF, Capacitor_SMD:C_0805_2012Metric, F.Cu at (-56.7, 150.1)
- added C38: 2.2uF, Capacitor_SMD:C_0805_2012Metric, F.Cu at (-81.4, 171.5)
- added C39: 100nF, Capacitor_SMD:C_0805_2012Metric, F.Cu at (-81.4, 174.5)
- added C40: 10nF, Capacitor_SMD:C_0805_2012Metric, F.Cu at (-81.4, 177.5)
- added C41: 100nF, Capacitor_SMD:C_0805_2012Metric, F.Cu at (-17.1, 88.5)
- added C42: 4.7uF, Capacitor_SMD:C_0805_2012Metric, F.Cu at (-19.8, 145.9)
- added C43: 100nF, Capacitor_SMD:C_0805_2012Metric, F.Cu at (-17.1, 91.5)
- added C44: 100nF, Capacitor_SMD:C_0805_2012Metric, F.Cu at (-17.1, 94.5)
- added C45: 100nF, Capacitor_SMD:C_0805_2012Metric, F.Cu at (-19.8, 148.9)
- added C46: 1uF, Capacitor_SMD:C_0805_2012Metric, F.Cu at (-19.8, 151.9)
- added C47: 100nF, Capacitor_SMD:C_0805_2012Metric, F.Cu at (-19.8, 154.9)
- added C48: 1uF, Capacitor_SMD:C_0805_2012Metric, F.Cu at (-80.6, 152.9)
- added C49: 100nF, Capacitor_SMD:C_0805_2012Metric, F.Cu at (-64.4, 128.5)
- added C50: 100nF, Capacitor_SMD:C_0805_2012Metric, F.Cu at (-80.6, 155.9)
- added C51: 10nF, Capacitor_SMD:C_0805_2012Metric, F.Cu at (-80.6, 158.9)
- added C52: 100nF, Capacitor_SMD:C_0805_2012Metric, F.Cu at (-80.6, 161.9)
- added C53: 100nF, Capacitor_SMD:C_0805_2012Metric, F.Cu at (-76.2, 152.9)
- added C54: 1uF, Capacitor_SMD:C_0805_2012Metric, F.Cu at (-76.2, 155.9)
- added C55: 1uF, Capacitor_SMD:C_0805_2012Metric, F.Cu at (-17.1, 97.5)
- added C56: 100nF, Capacitor_SMD:C_0805_2012Metric, F.Cu at (-19.8, 157.9)
- added C57: 1uF, Capacitor_SMD:C_0805_2012Metric, F.Cu at (-19.8, 160.9)
- added C58: 1uF, Capacitor_SMD:C_0805_2012Metric, F.Cu at (-22.8, 129.5)
- added C59: 100nF, Capacitor_SMD:C_0805_2012Metric, F.Cu at (-8.55, 145.9)
- added C60: 47nF, Capacitor_SMD:C_0805_2012Metric, F.Cu at (-8.55, 148.9)
- added C61: 10uF/10V, Capacitor_Tantalum_SMD:CP_EIA-3216-10_Kemet-I, F.Cu at (-73.9, 165.0)
- added C62: 100nF, Capacitor_SMD:C_0805_2012Metric, F.Cu at (-76.2, 158.9)
- added C63: 100pF, Capacitor_SMD:C_0805_2012Metric, F.Cu at (-8.55, 151.9)
- added C64: 100pF, Capacitor_SMD:C_0805_2012Metric, F.Cu at (-8.55, 154.9)
- added C65: 4.7nF, Capacitor_SMD:C_0805_2012Metric, F.Cu at (-8.55, 157.9)
- added C66: 100nF, Capacitor_SMD:C_0805_2012Metric, F.Cu at (-22.8, 132.5)
- added C67: 100nF, Capacitor_SMD:C_0805_2012Metric, F.Cu at (-76.2, 161.9)
- added C68: 1uF, Capacitor_SMD:C_0805_2012Metric, F.Cu at (-8.55, 160.9)
- added C69: 1uF, Capacitor_SMD:C_0805_2012Metric, F.Cu at (-71.7, 152.9)
- added C70: 100nF, Capacitor_SMD:C_0805_2012Metric, F.Cu at (-71.7, 155.9)
- added C71: 100nF, Capacitor_SMD:C_0805_2012Metric, F.Cu at (-71.7, 158.9)
- added C72: 1uF, Capacitor_SMD:C_0805_2012Metric, F.Cu at (-71.7, 161.9)
- added C73: 10uF, Capacitor_SMD:C_0805_2012Metric, F.Cu at (-64.4, 131.5)
- added C74: 1uF, Capacitor_SMD:C_0805_2012Metric, F.Cu at (-64.4, 134.5)
- added C75: 100nF, Capacitor_SMD:C_0805_2012Metric, F.Cu at (-22.8, 135.5)
- added C76: 100nF, Capacitor_SMD:C_0805_2012Metric, F.Cu at (-26.3, 145.9)
- added C77: 100uF/6.3V, Capacitor_Tantalum_SMD:CP_EIA-3528-12_Kemet-T, F.Cu at (-66.5, 162.3)
- added D1: LED, LED_SMD:LED_0805_2012Metric, F.Cu at (-14.1, 138.4)
- added D10: PESD3V3X1BL,315, PESD3V3X1BL:PESD5V0S1BL315, F.Cu at (-73.2, 121.3)
- added D11: PESD3V3X1BL,315, PESD3V3X1BL:PESD5V0S1BL315, F.Cu at (-73.2, 124.1)
- added D12: PESD3V3X1BL,315, PESD3V3X1BL:PESD5V0S1BL315, F.Cu at (-73.2, 126.9)
- added D13: PESD3V3X1BL,315, PESD3V3X1BL:PESD5V0S1BL315, F.Cu at (-73.2, 129.7)
- added D14: PESD3V3X1BL,315, PESD3V3X1BL:PESD5V0S1BL315, F.Cu at (-73.2, 132.5)
- added D15: PESD3V3X1BL,315, PESD3V3X1BL:PESD5V0S1BL315, F.Cu at (-16.1, 169.4)
- added D16: PESD3V3X1BL,315, PESD3V3X1BL:PESD5V0S1BL315, F.Cu at (-16.1, 172.2)
- added D17: PESD3V3X1BL,315, PESD3V3X1BL:PESD5V0S1BL315, F.Cu at (-16.1, 175.0)
- added D18: PESD3V3X1BL,315, PESD3V3X1BL:PESD5V0S1BL315, F.Cu at (-16.1, 177.8)
- added D19: PESD3V3X1BL,315, PESD3V3X1BL:PESD5V0S1BL315, F.Cu at (-40.1, 92.0)
- added D2: LED, LED_SMD:LED_0805_2012Metric, F.Cu at (-60.0, 128.5)
- added D20: PESD3V3X1BL,315, PESD3V3X1BL:PESD5V0S1BL315, F.Cu at (-40.1, 94.8)
- added D21: PESD3V3X1BL,315, PESD3V3X1BL:PESD5V0S1BL315, F.Cu at (-40.1, 97.5)
- added D22: PESD3V3X1BL,315, PESD3V3X1BL:PESD5V0S1BL315, F.Cu at (-40.1, 100.3)
- added D23: PESD3V3X1BL,315, PESD3V3X1BL:PESD5V0S1BL315, F.Cu at (-40.1, 103.2)
- added D24: PESD3V3X1BL,315, PESD3V3X1BL:PESD5V0S1BL315, F.Cu at (-37.0, 92.0)
- added D25: PESD3V3X1BL,315, PESD3V3X1BL:PESD5V0S1BL315, F.Cu at (-37.0, 94.8)
- added D26: PESD3V3X1BL,315, PESD3V3X1BL:PESD5V0S1BL315, F.Cu at (-37.0, 97.5)
- added D27: PESD3V3X1BL,315, PESD3V3X1BL:PESD5V0S1BL315, F.Cu at (-3.76, 135.5)
- added D28: PESD3V3X1BL,315, PESD3V3X1BL:PESD5V0S1BL315, F.Cu at (-3.76, 138.3)
- added D29: PESD3V3X1BL,315, PESD3V3X1BL:PESD5V0S1BL315, F.Cu at (-66.3, 174.9)
- added D3: LED, LED_SMD:LED_0805_2012Metric, F.Cu at (-60.0, 131.6)
- added D30: PESD3V3X1BL,315, PESD3V3X1BL:PESD5V0S1BL315, F.Cu at (-66.3, 177.7)
- added D31: PESD3V3X1BL,315, PESD3V3X1BL:PESD5V0S1BL315, F.Cu at (-52.9, 169.0)
- added D32: PESD3V3X1BL,315, PESD3V3X1BL:PESD5V0S1BL315, F.Cu at (-52.9, 171.8)
- added D33: PESD3V3X1BL,315, PESD3V3X1BL:PESD5V0S1BL315, F.Cu at (-3.86, 169.4)
- added D34: PESD3V3X1BL,315, PESD3V3X1BL:PESD5V0S1BL315, F.Cu at (-3.86, 172.2)
- added D35: PESD3V3X1BL,315, PESD3V3X1BL:PESD5V0S1BL315, F.Cu at (-3.86, 175.0)
- added D36: PESD3V3X1BL,315, PESD3V3X1BL:PESD5V0S1BL315, F.Cu at (-3.86, 177.8)
- added D37: PTVS6V0S1UR,115, PTVS6V0S1UR:SOD123W, F.Cu at (-63.6, 145.8)
- added D38: PESD3V3X1BL,315, PESD3V3X1BL:PESD5V0S1BL315, F.Cu at (-3.76, 121.1)
- added D39: PESD3V3X1BL,315, PESD3V3X1BL:PESD5V0S1BL315, F.Cu at (-3.76, 123.9)
- added D4: LED, LED_SMD:LED_0805_2012Metric, F.Cu at (-64.2, 148.8)
- added D40: PESD3V3X1BL,315, PESD3V3X1BL:PESD5V0S1BL315, F.Cu at (-3.76, 126.7)
- added D5: LED, LED_SMD:LED_0805_2012Metric, F.Cu at (-49.1, 158.7)
- added D6: PESD3V3X1BL,315, PESD3V3X1BL:PESD5V0S1BL315, F.Cu at (-57.3, 158.6)
- added D7: PESD3V3X1BL,315, PESD3V3X1BL:PESD5V0S1BL315, F.Cu at (-57.3, 161.4)
- added D8: PESD3V3X1BL,315, PESD3V3X1BL:PESD5V0S1BL315, F.Cu at (-57.3, 164.2)
- added D9: LED, LED_SMD:LED_0805_2012Metric, F.Cu at (-26.3, 148.9)
- added FB1: 1K/0.1A, Inductor_SMD:L_0603_1608Metric, F.Cu at (-49.3, 161.5)
- added FB2: 1K/0.1A, Inductor_SMD:L_0603_1608Metric, F.Cu at (-48.0, 146.0)
- added FB3: 1K/0.1A, Inductor_SMD:L_0603_1608Metric, F.Cu at (-77.1, 176.0)
- added FB4: 1K/0.1A, Inductor_SMD:L_0603_1608Metric, F.Cu at (-8.48, 99.6)
- added FB5: 1K/0.1A, Inductor_SMD:L_0603_1608Metric, F.Cu at (-15.6, 159.0)
- added FB6: 60R/6A, Inductor_SMD:L_1806_4516Metric, F.Cu at (-66.0, 166.2)
- added IC1: MX25L51245GXDI-08G, MX25L51245GZ:BGA24C100P5X5_600X800X120, F.Cu at (-37.2, 172.0)
- added IC2: ICP-10125, ICP-10125:ICP10125, F.Cu at (-7.17, 95.0)
- added IC4: EMIF06-HSD03F3, EMIF06-HSD03F3:EMIF06HSD03F3, F.Cu at (-18.4, 139.6)
- added J1: Micro_SD_Card_Det_Hirose_DM3AT, Connector_Card:microSD_HC_Hirose_DM3AT-SF-PEJM5, F.Cu at (-33.4, 125.5)
- added J10: SWDIO, Connector_Wire:SolderWirePad_1x01_SMD_1x2mm, F.Cu at (-57.6, 155.4)
- added J11: SWCLK, Connector_Wire:SolderWirePad_1x01_SMD_1x2mm, F.Cu at (-55.1, 155.4)
- added J12: SWO, Connector_Wire:SolderWirePad_1x01_SMD_1x2mm, F.Cu at (-52.5, 155.4)
- added J13: VCC, Connector_Wire:SolderWirePad_1x01_SMD_1x2mm, F.Cu at (-50.0, 155.4)
- added J14: GND, Connector_Wire:SolderWirePad_1x01_SMD_1x2mm, F.Cu at (-47.4, 155.4)
- added J15: VBUS, Connector_Wire:SolderWirePad_1x01_SMD_1x2mm, F.Cu at (-62.8, 125.2)
- added J16: DN, Connector_Wire:SolderWirePad_1x01_SMD_1x2mm, F.Cu at (-60.3, 125.2)
- added J17: DP, Connector_Wire:SolderWirePad_1x01_SMD_1x2mm, F.Cu at (-57.7, 125.2)
- added J18: GND, Connector_Wire:SolderWirePad_1x01_SMD_1x2mm, F.Cu at (-55.2, 125.2)
- added J19: GND, Connector_Wire:SolderWirePad_1x01_SMD_1.5x3mm, F.Cu at (1.29, 146.6)
- added J2: CAN_H, Connector_Wire:SolderWirePad_1x01_SMD_1.5x3mm, F.Cu at (-4.80, 146.6)
- added J20: GND, Connector_Wire:SolderWirePad_1x01_SMD_1.5x3mm, F.Cu at (-81.3, 165.7)
- added J21: +5V, Connector_Wire:SolderWirePad_1x01_SMD_1.5x3mm, F.Cu at (-78.3, 165.7)
- added J23: USB_C_Receptacle_USB2.0_16P, Connector_USB:USB_C_Receptacle_GCT_USB4085, F.Cu at (-38.9, 154.8)
- added J3: CAN_L, Connector_Wire:SolderWirePad_1x01_SMD_1.5x3mm, F.Cu at (-1.75, 146.6)
- added J4: DTR, Connector_Wire:SolderWirePad_1x01_SMD_1x2mm, F.Cu at (-65.4, 121.7)
- added J43: M, Connector_Wire:SolderWirePad_1x01_SMD_1x2mm, F.Cu at (-18.1, 104.6)
- added J47: C, Connector_Wire:SolderWirePad_1x01_SMD_1x2mm, F.Cu at (-15.5, 104.6)
- added J48: F, Connector_Wire:SolderWirePad_1x01_SMD_1x2mm, F.Cu at (-13.0, 104.6)
- added J49: D, Connector_Wire:SolderWirePad_1x01_SMD_1x2mm, F.Cu at (-10.4, 104.6)
- added J5: TXD, Connector_Wire:SolderWirePad_1x01_SMD_1x2mm, F.Cu at (-62.8, 121.7)
- added J50: SM1, Connector_Wire:SolderWirePad_1x01_SMD_1x2mm, F.Cu at (-8.49, 117.9)
- added J51: SM2, Connector_Wire:SolderWirePad_1x01_SMD_1x2mm, F.Cu at (-5.95, 117.9)
- added J52: SM3, Connector_Wire:SolderWirePad_1x01_SMD_1x2mm, F.Cu at (-3.40, 117.9)
- added J53: L1, Connector_Wire:SolderWirePad_1x01_SMD_1x2mm, F.Cu at (-8.60, 166.2)
- added J54: L2, Connector_Wire:SolderWirePad_1x01_SMD_1x2mm, F.Cu at (-6.04, 166.2)
- added J55: L3, Connector_Wire:SolderWirePad_1x01_SMD_1x2mm, F.Cu at (-3.50, 166.2)
- added J56: L4, Connector_Wire:SolderWirePad_1x01_SMD_1x2mm, F.Cu at (-0.94, 166.2)
- added J57: SCL, Connector_Wire:SolderWirePad_1x01_SMD_1x2mm, F.Cu at (-53.2, 175.0)
- added J58: SDA, Connector_Wire:SolderWirePad_1x01_SMD_1x2mm, F.Cu at (-50.7, 175.0)
- added J59: S1, Connector_Wire:SolderWirePad_1x01_SMD_1x2mm, F.Cu at (-71.1, 171.8)
- added J6: RXD, Connector_Wire:SolderWirePad_1x01_SMD_1x2mm, F.Cu at (-60.3, 121.7)
- added J60: S2, Connector_Wire:SolderWirePad_1x01_SMD_1x2mm, F.Cu at (-68.5, 171.8)
- added J61: TX/CH1, Connector_Wire:SolderWirePad_1x01_SMD_1x2mm, F.Cu at (-8.49, 132.3)
- added J62: RX/CH2, Connector_Wire:SolderWirePad_1x01_SMD_1x2mm, F.Cu at (-5.95, 132.3)
- added J63: T1, Connector_Wire:SolderWirePad_1x01_SMD_1x2mm, F.Cu at (-40.5, 88.8)
- added J64: R1, Connector_Wire:SolderWirePad_1x01_SMD_1x2mm, F.Cu at (-37.9, 88.8)
- added J65: T2, Connector_Wire:SolderWirePad_1x01_SMD_1x2mm, F.Cu at (-35.4, 88.8)
- added J66: R2, Connector_Wire:SolderWirePad_1x01_SMD_1x2mm, F.Cu at (-32.8, 88.8)
- added J67: T3, Connector_Wire:SolderWirePad_1x01_SMD_1x2mm, F.Cu at (-30.3, 88.8)
- added J68: R3, Connector_Wire:SolderWirePad_1x01_SMD_1x2mm, F.Cu at (-27.7, 88.8)
- added J69: T4, Connector_Wire:SolderWirePad_1x01_SMD_1x2mm, F.Cu at (-25.2, 88.8)
- added J7: VCC, Connector_Wire:SolderWirePad_1x01_SMD_1x2mm, F.Cu at (-57.7, 121.7)
- added J70: R4, Connector_Wire:SolderWirePad_1x01_SMD_1x2mm, F.Cu at (-22.6, 88.8)
- added J71: M1, Connector_Wire:SolderWirePad_1x01_SMD_1x2mm, F.Cu at (-20.8, 166.2)
- added J72: M2, Connector_Wire:SolderWirePad_1x01_SMD_1x2mm, F.Cu at (-18.2, 166.2)
- added J73: M3, Connector_Wire:SolderWirePad_1x01_SMD_1x2mm, F.Cu at (-15.7, 166.2)
- added J74: M4, Connector_Wire:SolderWirePad_1x01_SMD_1x2mm, F.Cu at (-13.1, 166.2)
- added J8: GND, Connector_Wire:SolderWirePad_1x01_SMD_1x2mm, F.Cu at (-55.2, 121.7)
- added J9: RTS, Connector_Wire:SolderWirePad_1x01_SMD_1x2mm, F.Cu at (-65.4, 125.2)
- added L1: 74438334015, WE-74438334015:INDC3030X120N, F.Cu at (-63.7, 142.0)
- added NT1: Tie_MCU_Rail, NetTie:NetTie-2_SMD_Pad0.5mm, F.Cu at (-50.0, 163.5)
- added NT2: Tie_FLASH_Rail, NetTie:NetTie-2_SMD_Pad0.5mm, F.Cu at (-40.5, 178.3)
- added NT3: Tie_IMU_1_Rail, NetTie:NetTie-2_SMD_Pad0.5mm, F.Cu at (-48.8, 148.0)
- added NT4: Tie_IMU_2_Rail, NetTie:NetTie-2_SMD_Pad0.5mm, F.Cu at (-77.9, 178.0)
- added NT5: Tie_MAG_Rail, NetTie:NetTie-2_SMD_Pad0.5mm, F.Cu at (-16.4, 161.0)
- added Q1: FDN340P, Package_TO_SOT_SMD:SOT-23, F.Cu at (-18.1, 130.2)
- added Q2: BC847, Package_TO_SOT_SMD:SOT-23, F.Cu at (-18.1, 134.6)
- added Q3: BC847BDW1, Package_TO_SOT_SMD:SOT-363_SC-70-6, F.Cu at (-60.2, 134.9)
- added Q4: BC847, Package_TO_SOT_SMD:SOT-23, F.Cu at (-69.1, 122.1)
- added Q5: FDN340P, Package_TO_SOT_SMD:SOT-23, F.Cu at (-69.1, 126.6)
- added Q6: BC847BDW1, Package_TO_SOT_SMD:SOT-363_SC-70-6, F.Cu at (-68.4, 141.4)
- added Q7: BC847BDW1, Package_TO_SOT_SMD:SOT-363_SC-70-6, F.Cu at (-68.4, 144.9)
- added Q8: BC847, Package_TO_SOT_SMD:SOT-23, F.Cu at (-69.1, 131.0)
- added Q9: BC847, Package_TO_SOT_SMD:SOT-23, F.Cu at (-27.7, 160.0)
- added R10: 10K, Resistor_SMD:R_0805_2012Metric, F.Cu at (-30.4, 179.9)
- added R100: 22R, Resistor_SMD:R_0805_2012Metric, F.Cu at (-7.67, 169.4)
- added R101: 22R, Resistor_SMD:R_0805_2012Metric, F.Cu at (-7.67, 172.4)
- added R102: 22R, Resistor_SMD:R_0805_2012Metric, F.Cu at (-7.67, 175.3)
- added R103: 22R, Resistor_SMD:R_0805_2012Metric, F.Cu at (-7.67, 178.3)
- added R105: 22R, Resistor_SMD:R_0805_2012Metric, F.Cu at (-7.57, 121.2)
- added R106: 22R, Resistor_SMD:R_0805_2012Metric, F.Cu at (-7.57, 124.1)
- added R107: 22R, Resistor_SMD:R_0805_2012Metric, F.Cu at (-7.57, 127.1)
- added R11: 10K, Resistor_SMD:R_0805_2012Metric, F.Cu at (-52.3, 146.2)
- added R12: 10K, Resistor_SMD:R_0805_2012Metric, F.Cu at (-52.3, 149.1)
- added R13: 10K, Resistor_SMD:R_0805_2012Metric, F.Cu at (-85.8, 171.5)
- added R14: 3.3K, Resistor_SMD:R_0805_2012Metric, F.Cu at (-85.8, 174.4)
- added R15: 3.3K, Resistor_SMD:R_0805_2012Metric, F.Cu at (-85.8, 177.4)
- added R16: 3.3K, Resistor_SMD:R_0805_2012Metric, F.Cu at (-85.8, 180.3)
- added R17: 3.3K, Resistor_SMD:R_0805_2012Metric, F.Cu at (-12.7, 88.5)
- added R18: 3.3K, Resistor_SMD:R_0805_2012Metric, F.Cu at (-12.7, 91.4)
- added R19: 3.3K, Resistor_SMD:R_0805_2012Metric, F.Cu at (-12.7, 94.4)
- added R20: 3.3K, Resistor_SMD:R_0805_2012Metric, F.Cu at (-12.7, 97.3)
- added R21: 3.3K, Resistor_SMD:R_0805_2012Metric, F.Cu at (-15.4, 145.8)
- added R22: 3.3K, Resistor_SMD:R_0805_2012Metric, F.Cu at (-15.4, 148.8)
- added R23: 10K, Resistor_SMD:R_0805_2012Metric, F.Cu at (-15.4, 151.7)
- added R24: 10K, Resistor_SMD:R_0805_2012Metric, F.Cu at (-85.8, 141.1)
- added R25: 10K, Resistor_SMD:R_0805_2012Metric, F.Cu at (-85.8, 144.0)
- added R26: 47K, Resistor_SMD:R_0805_2012Metric, F.Cu at (-22.8, 117.6)
- added R27: 47K, Resistor_SMD:R_0805_2012Metric, F.Cu at (-22.8, 120.6)
- added R28: 47K, Resistor_SMD:R_0805_2012Metric, F.Cu at (-22.8, 123.5)
- added R29: 47K, Resistor_SMD:R_0805_2012Metric, F.Cu at (-22.8, 126.5)
- added R30: 47K, Resistor_SMD:R_0805_2012Metric, F.Cu at (-18.4, 117.6)
- added R31: 47K, Resistor_SMD:R_0805_2012Metric, F.Cu at (-18.4, 120.6)
- added R32: 47K, Resistor_SMD:R_0805_2012Metric, F.Cu at (-18.4, 123.5)
- added R33: 10K, Resistor_SMD:R_0805_2012Metric, F.Cu at (-18.4, 126.5)
- added R34: 10K, Resistor_SMD:R_0805_2012Metric, F.Cu at (-14.0, 117.6)
- added R35: 1K, Resistor_SMD:R_0805_2012Metric, F.Cu at (-14.0, 120.6)
- added R36: 470R, Resistor_SMD:R_0805_2012Metric, F.Cu at (-14.0, 123.5)
- added R37: 10K, Resistor_SMD:R_0805_2012Metric, F.Cu at (-85.8, 147.0)
- added R38: 1.3K, Resistor_SMD:R_0805_2012Metric, F.Cu at (-4.12, 150.4)
- added R39: 1.3K, Resistor_SMD:R_0805_2012Metric, F.Cu at (-4.12, 153.3)
- added R40: 75K, Resistor_SMD:R_0805_2012Metric, F.Cu at (-85.8, 149.9)
- added R41: 24K, Resistor_SMD:R_0805_2012Metric, F.Cu at (-81.4, 141.1)
- added R42: 100R, Resistor_SMD:R_0805_2012Metric, F.Cu at (-81.4, 144.0)
- added R43: 10K, Resistor_SMD:R_0805_2012Metric, F.Cu at (-85.8, 121.4)
- added R44: 10K, Resistor_SMD:R_0805_2012Metric, F.Cu at (-85.8, 124.3)
- added R45: 10K, Resistor_SMD:R_0805_2012Metric, F.Cu at (-85.8, 127.3)
- added R46: 10K, Resistor_SMD:R_0805_2012Metric, F.Cu at (-85.8, 130.2)
- added R47: 10K, Resistor_SMD:R_0805_2012Metric, F.Cu at (-85.8, 133.2)
- added R48: 470R, Resistor_SMD:R_0805_2012Metric, F.Cu at (-85.8, 136.1)
- added R49: 1K, Resistor_SMD:R_0805_2012Metric, F.Cu at (-81.4, 121.4)
- added R50: 47K, Resistor_SMD:R_0805_2012Metric, F.Cu at (-81.4, 124.3)
- added R51: 10K, Resistor_SMD:R_0805_2012Metric, F.Cu at (-81.4, 127.3)
- added R52: 10K, Resistor_SMD:R_0805_2012Metric, F.Cu at (-81.4, 130.2)
- added R53: 470R, Resistor_SMD:R_0805_2012Metric, F.Cu at (-81.4, 133.2)
- added R54: 470R, Resistor_SMD:R_0805_2012Metric, F.Cu at (-53.5, 158.7)
- added R55: 1K, Resistor_SMD:R_0805_2012Metric, F.Cu at (-81.4, 147.0)
- added R56: 1K, Resistor_SMD:R_0805_2012Metric, F.Cu at (-81.4, 149.9)
- added R57: 1K, Resistor_SMD:R_0805_2012Metric, F.Cu at (-77.0, 141.1)
- added R58: 10K, Resistor_SMD:R_0805_2012Metric, F.Cu at (-77.0, 144.0)
- added R59: 1K, Resistor_SMD:R_0805_2012Metric, F.Cu at (-77.0, 147.0)
- added R60: 1K, Resistor_SMD:R_0805_2012Metric, F.Cu at (-77.0, 149.9)
- added R61: 470R, Resistor_SMD:R_0805_2012Metric, F.Cu at (-39.5, 145.8)
- added R62: 0R, Resistor_SMD:R_0805_2012Metric, F.Cu at (-39.5, 148.8)
- added R63: 5.1K, Resistor_SMD:R_0805_2012Metric, F.Cu at (-39.5, 151.7)
- added R64: 5.1K, Resistor_SMD:R_0805_2012Metric, F.Cu at (-35.1, 145.8)
- added R65: 33K, Resistor_SMD:R_0805_2012Metric, F.Cu at (-35.1, 148.8)
- added R66: 82K, Resistor_SMD:R_0805_2012Metric, F.Cu at (-35.1, 151.7)
- added R67: 1K, Resistor_SMD:R_0805_2012Metric, F.Cu at (-81.4, 136.1)
- added R68: 10K, Resistor_SMD:R_0805_2012Metric, F.Cu at (-77.0, 121.4)
- added R69: 0R, Resistor_SMD:R_0805_2012Metric, F.Cu at (-77.0, 124.3)
- added R70: 0R, Resistor_SMD:R_0805_2012Metric, F.Cu at (-77.0, 127.3)
- added R71: 0R, Resistor_SMD:R_0805_2012Metric, F.Cu at (-53.5, 161.6)
- added R72: 10K, Resistor_SMD:R_0805_2012Metric, F.Cu at (-72.6, 141.1)
- added R73: 10K, Resistor_SMD:R_0805_2012Metric, F.Cu at (-72.6, 144.0)
- added R74: 10K, Resistor_SMD:R_0805_2012Metric, F.Cu at (-72.6, 147.0)
- added R75: 10K, Resistor_SMD:R_0805_2012Metric, F.Cu at (-72.6, 149.9)
- added R76: 10K, Resistor_SMD:R_0805_2012Metric, F.Cu at (-30.7, 145.8)
- added R77: 1K, Resistor_SMD:R_0805_2012Metric, F.Cu at (-30.7, 148.8)
- added R78: 22R, Resistor_SMD:R_0805_2012Metric, F.Cu at (-19.9, 169.4)
- added R79: 22R, Resistor_SMD:R_0805_2012Metric, F.Cu at (-19.9, 172.4)
- added R80: 22R, Resistor_SMD:R_0805_2012Metric, F.Cu at (-19.9, 175.3)
- added R81: 22R, Resistor_SMD:R_0805_2012Metric, F.Cu at (-19.9, 178.3)
- added R82: 47K, Resistor_SMD:R_0805_2012Metric, F.Cu at (-14.0, 126.5)
- added R83: 0R, Resistor_SMD:R_0805_2012Metric, F.Cu at (-30.7, 151.7)
- added R84: 22R, Resistor_SMD:R_0805_2012Metric, F.Cu at (-33.1, 92.0)
- added R85: 22R, Resistor_SMD:R_0805_2012Metric, F.Cu at (-33.1, 95.0)
- added R86: 22R, Resistor_SMD:R_0805_2012Metric, F.Cu at (-33.1, 97.9)
- added R87: 22R, Resistor_SMD:R_0805_2012Metric, F.Cu at (-33.1, 100.9)
- added R88: 22R, Resistor_SMD:R_0805_2012Metric, F.Cu at (-33.1, 103.8)
- added R89: 22R, Resistor_SMD:R_0805_2012Metric, F.Cu at (-33.1, 106.8)
- added R9: 10K, Resistor_SMD:R_0805_2012Metric, F.Cu at (-30.4, 176.9)
- added R90: 22R, Resistor_SMD:R_0805_2012Metric, F.Cu at (-33.1, 109.7)
- added R91: 22R, Resistor_SMD:R_0805_2012Metric, F.Cu at (-33.1, 112.7)
- added R92: 22R, Resistor_SMD:R_0805_2012Metric, F.Cu at (-7.57, 135.6)
- added R93: 22R, Resistor_SMD:R_0805_2012Metric, F.Cu at (-7.57, 138.5)
- added R94: 22R, Resistor_SMD:R_0805_2012Metric, F.Cu at (-70.1, 175.0)
- added R95: 22R, Resistor_SMD:R_0805_2012Metric, F.Cu at (-70.1, 178.0)
- added R96: 22R, Resistor_SMD:R_0805_2012Metric, F.Cu at (-56.7, 169.1)
- added R97: 22R, Resistor_SMD:R_0805_2012Metric, F.Cu at (-56.7, 172.0)
- added R98: 10K, Resistor_SMD:R_0805_2012Metric, F.Cu at (-56.7, 175.0)
- added R99: 10K, Resistor_SMD:R_0805_2012Metric, F.Cu at (-56.7, 177.9)
- added TP1: VDDBLE, TestPoint:TestPoint_Pad_D1.5mm, F.Cu at (-56.0, 128.8)
- added U1: BMI088, Package_LGA:Bosch_LGA-16_4.5x3mm_P0.5mm_LayoutBorder7x1y_ClockwisePinNumbering, F.Cu at (-51.3, 142.3)
- added U10: NCP163ASN180T1G, Package_TO_SOT_SMD:SOT-23-5, F.Cu at (-85.4, 158.4)
- added U11: NCP163ASN330T1G, Package_TO_SOT_SMD:SOT-23-5, F.Cu at (-85.4, 163.1)
- added U12: USBLC6-2SC6, Package_TO_SOT_SMD:SOT-23-6, F.Cu at (-27.6, 155.6)
- added U4: ICM-40609-D, ICM-40609-D:ICM-40609-D, F.Cu at (-76.5, 172.6)
- added U5: IST8310, Package_LGA:LGA-16_3x3mm_P0.5mm, F.Cu at (-15.0, 155.5)
- added U6: TCA9517ADGK, Package_SO:VSSOP-8_3x3mm_P0.65mm, F.Cu at (-6.79, 89.4)
- added U7: AP62300WU, Package_TO_SOT_SMD:TSOT-23-6, F.Cu at (-85.4, 153.8)
- added U8: TJA1051TK-3, Package_SON:HVSON-8-1EP_3x3mm_P0.65mm_EP1.6x2.4mm, F.Cu at (-3.30, 157.1)
- added U9: ESP32-C6-MINI-1, RF_Module:ESP32-C6-MINI-1, F.Cu at (-65.9, 113.5)
- R1: value 220R -> 1K
- moved U3 3.61 mm to (-66.8, 70.2)
Connections:
- C22 pad 2: VDDUSB -> VDDMCU
- C23 pad 2: VDDUSB -> VDDMCU
- R1 pad 1: unconnected-(R1-Pad1) -> +5V
- S1 pad MP1: Net-(C16-Pad2) -> GND
- S1 pad MP2: Net-(C16-Pad2) -> GND
- S2 pad MP1: Net-(C17-Pad2) -> GND
- S2 pad MP2: Net-(C17-Pad2) -> GND
- U3 pad A10: unconnected-(U3-PA15(JTDI)-PadA10) -> /BLE/BLE_CTS
- U3 pad A2: unconnected-(U3-PE3-PadA2) -> /MCU/SBUS_2
- U3 pad A3: unconnected-(U3-PE2-PadA3) -> /MCU/I2S MCK
- U3 pad A4: unconnected-(U3-PE1-PadA4) -> /T1
- U3 pad A5: unconnected-(U3-PE0-PadA5) -> /R1
- U3 pad A6: unconnected-(U3-PB4(NJTRST)-PadA6) -> /MCU/SBUS_1
- U3 pad A8: unconnected-(U3-PD6-PadA8) -> /MCU/RX_RADIO
- U3 pad B10: unconnected-(U3-PC11-PadB10) -> /SD_Card/OUT_D3
- U3 pad B11: unconnected-(U3-PC10-PadB11) -> /SD_Card/OUT_D2
- U3 pad B2: unconnected-(U3-PE4-PadB2) -> /MCU/I2S FS
- U3 pad B3: unconnected-(U3-PE5-PadB3) -> /MCU/I2S SCK
- U3 pad B4: unconnected-(U3-PE6-PadB4) -> /CAN Tranciever/CAN_Sleep
- U3 pad B5: unconnected-(U3-PB9-PadB5) -> /CAN Tranciever/CAN_TX
- U3 pad B8: unconnected-(U3-PG12-PadB8) -> /MCU/SERVO 1
- U3 pad B9: unconnected-(U3-PD5-PadB9) -> /MCU/TX_RADIO
- U3 pad C10: unconnected-(U3-PC12-PadC10) -> /SD_Card/OUT_CLK
- U3 pad C11: VDDUSB -> VDDMCU
- U3 pad C3: unconnected-(U3-PF0-PadC3) -> /Barometer/SDA
- U3 pad C4: unconnected-(U3-PF1-PadC4) -> /Barometer/SCL
- U3 pad C5: unconnected-(U3-PB8-PadC5) -> /CAN Tranciever/CAN_RX
- U3 pad C6: unconnected-(U3-PB6-PadC6) -> /MCU/MAG_SCL
- U3 pad C7: unconnected-(U3-PG14-PadC7) -> /MCU/MAG_RST
- U3 pad D10: unconnected-(U3-PD1-PadD10) -> /BLE/BLE_RX
- U3 pad D11: unconnected-(U3-PA10-PadD11) -> /BLE/CHIP_PU
- U3 pad D12: unconnected-(U3-PA9-PadD12) -> /MCU/VBUS_SENSE
- U3 pad D4: unconnected-(U3-PF2-PadD4) -> /MCU/SERVO 2
- U3 pad D6: unconnected-(U3-PB7-PadD6) -> /MCU/MAG_SDA
- U3 pad D7: unconnected-(U3-PG13-PadD7) -> /MCU/MAG_INT
- U3 pad D9: unconnected-(U3-PD3-PadD9) -> /BLE/BLE_PW
- U3 pad E10: unconnected-(U3-PD0-PadE10) -> /BLE/BLE_TX
- U3 pad E11: unconnected-(U3-PC9-PadE11) -> /SD_Card/OUT_D1
- U3 pad E12: unconnected-(U3-PA8-PadE12) -> /SD_Card/uSD_Rail_Ctrl
- U3 pad E2: unconnected-(U3-PF3-PadE2) -> /MCU/SERVO 3
- U3 pad E9: unconnected-(U3-PD2-PadE9) -> /SD_Card/OUT_CMD
- U3 pad F11: unconnected-(U3-PC8-PadF11) -> /SD_Card/OUT_D0
- U3 pad F12: unconnected-(U3-PC7-PadF12) -> /R4
- U3 pad F2: unconnected-(U3-PF7-PadF2) -> /FLASH/OSPI_D2
- U3 pad F3: unconnected-(U3-PF6-PadF3) -> /FLASH/OSPI_D3
- U3 pad G1: unconnected-(U3-PF10-PadG1) -> /FLASH/OSPI_CLK
- U3 pad G11: unconnected-(U3-PG8-PadG11) -> /FLASH/FLASH_RST
- U3 pad G12: unconnected-(U3-PC6-PadG12) -> /T4
- U3 pad G2: unconnected-(U3-PF9-PadG2) -> /FLASH/OSPI_D1
- U3 pad G3: unconnected-(U3-PF8-PadG3) -> /FLASH/OSPI_D0
- U3 pad H11: unconnected-(U3-PG6-PadH11) -> /FLASH/OSPI_NCS
- U3 pad H12: unconnected-(U3-PG5-PadH12) -> /SD_Card/uSD_DET
- U3 pad H2: unconnected-(U3-PC1-PadH2) -> /MCU/I2S_SD
- U3 pad H8: unconnected-(U3-PE11-PadH8) -> /DSHOT/DSHOT_2
- U3 pad J2: unconnected-(U3-PA0-PadJ2) -> /IMU_1/CS_G
- U3 pad J3: unconnected-(U3-PA4-PadJ3) -> /IMU_1/CS_A
- U3 pad J4: unconnected-(U3-PC4-PadJ4) -> /IMU_1/INT
- U3 pad K10: unconnected-(U3-PD13-PadK10) -> /I2C/SDA
- U3 pad K11: unconnected-(U3-PD14-PadK11) -> /R2
- U3 pad K12: unconnected-(U3-PD15-PadK12) -> /T2
- U3 pad K3: unconnected-(U3-PA5-PadK3) -> /IMU_1/SCK
- U3 pad K5: unconnected-(U3-PF13-PadK5) -> /LEDs/NPXL 3
- U3 pad K7: unconnected-(U3-PE9-PadK7) -> /DSHOT/DSHOT_1
- U3 pad K8: unconnected-(U3-PE13-PadK8) -> /DSHOT/DSHOT_3
- U3 pad K9: unconnected-(U3-PD9-PadK9) -> /R3
- U3 pad L10: unconnected-(U3-PD12-PadL10) -> /I2C/SCL
- U3 pad L11: unconnected-(U3-PB14-PadL11) -> /IMU_2/SDO
- U3 pad L12: unconnected-(U3-PB15-PadL12) -> /IMU_2/MOSI
- U3 pad L3: unconnected-(U3-PA6-PadL3) -> /IMU_1/MISO
- U3 pad L4: unconnected-(U3-PB0-PadL4) -> /BLE/BLE_RTS
- U3 pad L5: unconnected-(U3-PF12-PadL5) -> /LEDs/NPXL 2
- U3 pad L8: unconnected-(U3-PE14-PadL8) -> /DSHOT/DSHOT_4
- U3 pad L9: unconnected-(U3-PD8-PadL9) -> /T3
- U3 pad M10: unconnected-(U3-PB11-PadM10) -> /IMU_2/INT2/FSYNC
- U3 pad M11: unconnected-(U3-PB12-PadM11) -> /IMU_2/nCS
- U3 pad M12: unconnected-(U3-PB13-PadM12) -> /IMU_2/SCLK
- U3 pad M3: unconnected-(U3-PA7-PadM3) -> /IMU_1/MOSI
- U3 pad M5: unconnected-(U3-PF11-PadM5) -> /LEDs/NPXL 1
- U3 pad M6: unconnected-(U3-PF14-PadM6) -> /LEDs/NPXL 4
- U3 pad M9: unconnected-(U3-PB10-PadM9) -> /IMU_2/INT1
Other:
- copper layers 2 -> 6
- rule pad_to_mask_clearance: 0 -> 0.1
