File: 141 FC.kicad_sch (KiCad schematic)
At the start: 0 parts

Commit message: Commit_1
Other:
- added sheet Barometer (ICP-10125.kicad_sch)
- added sheet FLASH (MX25L51245G.kicad_sch)
- added sheet IMU_1 (BMI088.kicad_sch)
- added sheet IMU_2 (ICM-40609-D.kicad_sch)
- added sheet Magnetometer (IST-8310.kicad_sch)

Commit message: progress
Other:
- added sheet BLE (ESP32C3.kicad_sch)
- added sheet CAN Tranciever (TJA1051.kicad_sch)
- added sheet Power_Distro (untitled.kicad_sch)
- added sheet SD_Card (SD_Card.kicad_sch)
Changed lines of the file:
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@@
 	)
 	(sheet
-		(at 185.42 88.9)
+		(at 116.84 54.61)
+		(size 12.7 12.7)
+		(exclude_from_sim no)
+		(in_bom yes)
+		(on_board yes)
+		(dnp no)
+		(fields_autoplaced yes)
+		(stroke
+			(width 0.1524)
+			(type solid)
+		)
+		(fill
+			(color 0 0 0 0)
+		)
+		(property "Sheetname" "BLE"
+			(at 116.84 53.8984 0)
+			(show_name no)
+			(do_not_autoplace no)
+			(effects
+				(font
+					(size 1.27 1.27)
+				)
+				(justify left bottom)
+			)
+		)
+		(property "Sheetfile" "ESP32C3.kicad_sch"
+			(at 116.84 67.8946 0)
+			(show_name no)
+			(do_not_autoplace no)
+			(effects
+				(font
+					(size 1.27 1.27)
+				)
+				(justify left top)
+			)
+		)
+		(instances
+			(project "141 FC"
+				(path "/524bae94-30c3-4d47-8232-d1fa64637976"
+					(page "11")
+				)
+			)
+		)
+	)
+	(sheet
+		(at 203.2 85.09)
 		(size 15.24 22.86)
 		(exclude_from_sim no)
@@
 		)
 		(property "Sheetname" "FLASH"
-			(at 185.42 88.1884 0)
+			(at 203.2 84.3784 0)
 			(show_name no)
 			(do_not_autoplace no)
@@
 		)
 		(property "Sheetfile" "MX25L51245G.kicad_sch"
-			(at 185.42 112.3446 0)
+			(at 203.2 108.5346 0)
 			(show_name no)
 			(do_not_autoplace no)
@@
 		)
 		(pin "OSPI_D2" bidirectional
-			(at 185.42 106.68 180)
+			(at 203.2 102.87 180)
 			(effects
 				(font
@@
 		)
 		(pin "OSPI_D3" bidirectional
-			(at 185.42 109.22 180)
+			(at 203.2 105.41 180)
 			(effects
 				(font
@@
 		)
 		(pin "OSPI_D0" bidirectional
-			(at 185.42 101.6 180)
+			(at 203.2 97.79 180)
 			(effects
 				(font
@@
 		)
 		(pin "OSPI_D1" bidirectional
-			(at 185.42 104.14 180)
+			(at 203.2 100.33 180)
 			(effects
 				(font
@@
 		)
 		(pin "OSPI_CLK" input
-			(at 185.42 99.06 180)
+			(at 203.2 95.25 180)
 			(effects
 				(font
@@
 		)
 		(pin "OSPI_NCS" input
-			(at 185.42 96.52 180)
+			(at 203.2 92.71 180)
 			(effects
 				(font
@@
 		)
 		(pin "FLASH_RST" input
-			(at 185.42 91.44 180)
+			(at 203.2 87.63 180)
 			(effects
 				(font
@@
 				)
 			)
+		)
+	)
+	(sheet
+		(at 88.9 30.48)
+		(size 12.7 12.7)
+		(exclude_from_sim no)
+		(in_bom yes)
+		(on_board yes)
+		(dnp no)
+		(fields_autoplaced yes)
+		(stroke
+			(width 0.1524)
+			(type solid)
+		)
+		(fill
+			(color 0 0 0 0)
+		)
+		(property "Sheetname" "Power_Distro"
+			(at 88.9 29.7684 0)
+			(show_name no)
+			(do_not_autoplace no)
+			(effects
+				(font
+					(size 1.27 1.27)
+				)
+				(justify left bottom)
+			)
+		)
+		(property "Sheetfile" "untitled.kicad_sch"
+			(at 88.9 43.7646 0)
+			(show_name no)
+			(do_not_autoplace no)
+			(effects
+				(font
+					(size 1.27 1.27)
+				)
+				(justify left top)
+			)
+		)
+		(instances
+			(project "141 FC"
+				(path "/524bae94-30c3-4d47-8232-d1fa64637976"
+					(page "8")
+				)
+			)
+		)
+	)
+	(sheet
+		(at 116.84 30.48)
+		(size 12.7 12.7)
+		(exclude_from_sim no)
+		(in_bom yes)
+		(on_board yes)
+		(dnp no)
+		(fields_autoplaced yes)
+		(stroke
+			(width 0.1524)
+			(type solid)
+		)
+		(fill
+			(color 0 0 0 0)
+		)
+		(property "Sheetname" "SD_Card"
+			(at 116.84 29.7684 0)
+			(show_name no)
+			(do_not_autoplace no)
+			(effects
+				(font
+					(size 1.27 1.27)
+				)
+				(justify left bottom)
+			)
+		)
+		(property "Sheetfile" "SD_Card.kicad_sch"
+			(at 116.84 43.7646 0)
+			(show_name no)
+			(do_not_autoplace no)
+			(effects
+				(font
+					(size 1.27 1.27)
+				)
+				(justify left top)
+			)
+		)
+		(instances
+			(project "141 FC"
+				(path "/524bae94-30c3-4d47-8232-d1fa64637976"
+					(page "9")
+				)
+			)
+		)
+	)
+	(sheet
+		(at 88.9 54.61)
+		(size 12.7 12.7)
+		(exclude_from_sim no)
+		(in_bom yes)
+		(on_board yes)
+		(dnp no)
+		(fields_autoplaced yes)
+		(stroke
+			(width 0.1524)
+			(type solid)
+		)
+		(fill
+			(color 0 0 0 0)
+		)
+		(property "Sheetname" "CAN Tranciever"
+			(at 88.9 53.8984 0)
+			(show_name no)
+			(do_not_autoplace no)
+			(effects
+				(font
+					(size 1.27 1.27)
+				)
+				(justify left bottom)
+			)
+		)
+		(property "Sheetfile" "TJA1051.kicad_sch"
+			(at 88.9 67.8946 0)
+			(show_name no)
+			(do_not_autoplace no)
+			(effects
+				(font
+					(size 1.27 1.27)
+				)
+				(justify left top)
+			)
+		)
+		(instances
+			(project "141 FC"
+				(path "/524bae94-30c3-4d47-8232-d1fa64637976"
+					(page "10")
+				)
+			)

Commit message: Almost Complete Schematic
Parts:
- added J43: M, Connector_Wire:SolderWirePad_1x01_SMD_1x2mm, symbol Connector:Conn_01x01_Pin
- added J47: C, Connector_Wire:SolderWirePad_1x01_SMD_1x2mm, symbol Connector:Conn_01x01_Pin
- added J48: F, Connector_Wire:SolderWirePad_1x01_SMD_1x2mm, symbol Connector:Conn_01x01_Pin
- added J49: D, Connector_Wire:SolderWirePad_1x01_SMD_1x2mm, symbol Connector:Conn_01x01_Pin
Connections:
- new net MCU/I2S FS: J48.1 (Pin_1)
- new net MCU/I2S MCK: J43.1 (Pin_1)
- new net MCU/I2S SCK: J47.1 (Pin_1)
- new net MCU/I2S_SD: J49.1 (Pin_1)
Other:
- added sheet DSHOT (untitled_1.kicad_sch)
- added sheet I2C (untitled_5.kicad_sch)
- added sheet LEDs (untitled_6.kicad_sch)
- added sheet RADIO (untitled_3.kicad_sch)
- added sheet SBUS (untitled_4.kicad_sch)
- added sheet SERVOs (untitled7.kicad_sch)
- added sheet UART (untitled_2.kicad_sch)
- added sheet USB_C_2.0 (USB_C_2.0.kicad_sch)
- sheet BLE ports: added BLE_CTS, BLE_PW, BLE_RST, BLE_RTS, BLE_RX, BLE_TX; removed none
- sheet CAN Tranciever ports: added CAN_RX, CAN_Sleep, CAN_TX; removed none
- sheet MCU ports: added BAR_SCL, BAR_SDA, BLE_CTS, BLE_POWER, BLE_RST, BLE_RTS, BLE_RX, BLE_TX, CAN_RX, CAN_SLEEP, CAN_TX, FLASH_RST, I2S FS, I2S MCK, I2S SCK, I2S_SD, IMU_1_INT, IMU_1_MISO, IMU_1_MOSI, IMU_1_SCK, IMU_1_nCS_A, IMU_1_nCS_G, IMU_2_INT_1, IMU_2_INT_2, IMU_2_MISO, IMU_2_MOSI, IMU_2_SCK, IMU_2_nCS, M1, M2, M3, M4, MAG_INT, MAG_RST, MAG_SCL, MAG_SDA, NEO PIXEL 1, NEO PIXEL 2, NEO PIXEL 3, NEO PIXEL 4, OSPI_CLK, OSPI_D0, OSPI_D1, OSPI_D2, OSPI_D3, OSPI_NCS, R1, R2, R3, R4, RX_RADIO, SBUS_1, SBUS_2, SCL, SDA, SD_CLK, SD_CMD, SD_D0, SD_D1, SD_D2, SD_D3, SD_DET, SD_PWR, SERVO 1, SERVO 2, SERVO 3, T1, T2, T3, T4, TX_RADIO, USB_DM, USB_DP, VBUS_SENSE; removed none
- sheet SD_Card ports: added SD_CK, SD_CMD, SD_D0, SD_D1, SD_D2, SD_D3, SD_DET, SD_EN; removed none
- note added: "Audio OUT"
