File: ESP32C3.kicad_sch (KiCad schematic)
At the start: 1 part, among them U9 ESP32-C6-MINI-1

Commit message: Almost Complete Schematic
Parts:
- added C49: 100nF, Capacitor_SMD:C_0805_2012Metric, symbol Device:C
- added C73: 10uF, Capacitor_SMD:C_0805_2012Metric, symbol Device:C
- added C74: 1uF, Capacitor_SMD:C_0805_2012Metric, symbol Device:C
- added D10, D11, D12, D13, D14: PESD3V3X1BL,315, PESD3V3X1BL:PESD5V0S1BL315, symbol PESD3V3X1BL_315:PESD3V3X1BL,315
- added D2, D3: LED, LED_SMD:LED_0805_2012Metric, symbol Device:LED
- added J15: VBUS, Connector_Wire:SolderWirePad_1x01_SMD_1x2mm, symbol Connector:Conn_01x01_Pin
- added J16: DN, Connector_Wire:SolderWirePad_1x01_SMD_1x2mm, symbol Connector:Conn_01x01_Pin
- added J17: DP, Connector_Wire:SolderWirePad_1x01_SMD_1x2mm, symbol Connector:Conn_01x01_Pin
- added J18, J8: GND, Connector_Wire:SolderWirePad_1x01_SMD_1x2mm, symbol Connector:Conn_01x01_Pin
- added J4: DTR, Connector_Wire:SolderWirePad_1x01_SMD_1x2mm, symbol Connector:Conn_01x01_Pin
- added J5: TXD, Connector_Wire:SolderWirePad_1x01_SMD_1x2mm, symbol Connector:Conn_01x01_Pin
- added J6: RXD, Connector_Wire:SolderWirePad_1x01_SMD_1x2mm, symbol Connector:Conn_01x01_Pin
- added J7: VCC, Connector_Wire:SolderWirePad_1x01_SMD_1x2mm, symbol Connector:Conn_01x01_Pin
- added J9: RTS, Connector_Wire:SolderWirePad_1x01_SMD_1x2mm, symbol Connector:Conn_01x01_Pin
- added Q3: BC847BDW1, Package_TO_SOT_SMD:SOT-363_SC-70-6, symbol Transistor_BJT:BC847BDW1
- added Q4, Q8: BC847, Package_TO_SOT_SMD:SOT-23, symbol Transistor_BJT:BC847
- added Q5: FDN340P, Package_TO_SOT_SMD:SOT-23, symbol Transistor_FET:FDN340P
- added R43, R44, R45, R46, R47, R51, R52, R68: 10K, Resistor_SMD:R_0805_2012Metric, symbol Device:R
- added R48, R53: 470R, Resistor_SMD:R_0805_2012Metric, symbol Device:R
- added R49, R67: 1K, Resistor_SMD:R_0805_2012Metric, symbol Device:R
- added R50: 47K, Resistor_SMD:R_0805_2012Metric, symbol Device:R
- added R69, R70: 0R, Resistor_SMD:R_0805_2012Metric, symbol Device:R
- added TP1: VDDBLE, TestPoint:TestPoint_Pad_D1.5mm, symbol Connector:TestPoint
Connections:
- net GND: now also C49.1, C73.1, C74.1, D10.2 (K2), D11.2 (K2), D12.2 (K2), D13.2 (K2), D14.2 (K2), D3.1 (K), J18.1 (Pin_1), J8.1 (Pin_1), Q4.2 (E), Q8.2 (E), R51.2
- net BLE_CTS: now reaches U9.10 (IO5)
- net BLE_RX: now reaches U9.15 (IO6)
- net BLE_TX: now reaches U9.16 (IO7)
- net DN: now reaches U9.17 (IO12)
- net DN: now also J16.1 (Pin_1)
- net DP: now reaches U9.18 (IO13)
- net DP: now also J17.1 (Pin_1)
- net VBUS_SENSE: now reaches U9.19 (IO14)
- net VBUS_SENSE: now also Q8.3 (C), R68.2
- net GPIO_8: now reaches U9.22 (IO8)
- net GPIO_8: now also D2.1 (K), R44.1
- net GPIO_9: now reaches U9.23 (IO9)
- net GPIO_9: now also Q3.3 (C2), R45.1
- net VDDBLE: now reaches U9.3 (3V3)
- net VDDBLE: now also C49.2, C73.2, Q5.3 (D), R43.2, R44.2, R45.2, R48.2, R53.1, R68.1, R69.1, R70.1, TP1.1
- net RXD: now reaches U9.30 (RXD0)
- net RXD: now also D12.1 (K1), J6.1 (Pin_1)
- net TXD: now reaches U9.31 (TXD0)
- net TXD: now also D13.1 (K1), J5.1 (Pin_1)
- net BLE_RST: now reaches U9.8 (EN)
- net BLE_RST: now also C74.2, Q3.6 (C1), R43.1
- net BLE_RTS: now reaches U9.9 (IO4)
- new net: Q3.2 (B1), R47.1
- new net: Q8.1 (B), R67.1
- new net: J15.1 (Pin_1), R67.2
- new net: Q3.5 (B2), R46.2
- new net: D11.1 (K1), J7.1 (Pin_1), R70.2
- new net: D3.2 (A), R53.2
- new net: Q4.1 (B), R49.2, R51.1
- new net: Q5.1 (G), R50.2, R52.1
- new net: D2.2 (A), R48.1
- new net: Q4.3 (C), R52.2
- new net BLE_PW: R49.1
- new net DTR: D14.1 (K1), J4.1 (Pin_1), Q3.4 (E2), R47.2
- new net RTS: D10.1 (K1), J9.1 (Pin_1), Q3.1 (E1), R46.1
- new net VDD: Q5.2 (S), R50.1, R69.2
- no-connect marks 0 -> 11
Other:
- note added: "Auto Download"
- note added: "By-Pass Capacitors"
- note added: "Chip Pull-Up"
- note added: "FLASH"
- note added: "LED_BUILT_IN"
- note added: "Populate R61 for BLE always ON & remove everything else."
- note added: "Power Tree"
- note added: "USB"
