File: ICM-40609-D.kicad_sch (KiCad schematic)
At the start: 8 parts, among them U4 ICM-40609-D

Commit message: progress
Parts:
- added FB3: 1K/0.1A, Inductor_SMD:L_0603_1608Metric, symbol Device:FerriteBead_Small
- added NT4: Tie_IMU_2_Rail, NetTie:NetTie-2_SMD_Pad0.5mm, symbol Device:NetTie_2
Connections:
- net VDDIMU_2: now also FB3.2; no longer C40.1, R13.1, R14.1, R15.1, R16.1, U4.8 (VDDIO)
- new net VDDIMU_2_IO: C40.1, FB3.1, NT4.2, R13.1, R14.1, R15.1, R16.1, U4.8 (VDDIO)
- new net VDD_3V3_S: NT4.1
Other:
- moved on the sheet: C38, C39, C40

Commit message: Almost Complete Schematic
Parts:
- R14, R15, R16: value 10K -> 3.3K
Changed lines of the file:
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@@
 			)
 		)
-		(property "Value" "10K"
+		(property "Value" "3.3K"
 			(at 121.92 54.61 90)
 			(show_name no)
@@
 			)
 		)
-		(property "Value" "10K"
+		(property "Value" "3.3K"
 			(at 102.87 54.61 90)
 			(show_name no)
@@
 			)
 		)
-		(property "Value" "10K"
+		(property "Value" "3.3K"
 			(at 113.03 54.61 90)
 			(show_name no)
