File: ICP-10125.kicad_sch (KiCad schematic)
At the start: 9 parts, among them IC2 ICP-10125, U6 TCA9517ADGK

Commit message: progress
Parts:
- added C55: 1uF, Capacitor_SMD:C_0805_2012Metric, symbol Device:C
- added FB4: 1K/0.1A, Inductor_SMD:L_0603_1608Metric, symbol Device:FerriteBead_Small
Connections:
- net GND: now also C55.1
- net VDDBAR: now also C55.2, FB4.1
- net VDDMCU renamed VDD
- new net VDD_1V8: FB4.2
Other:
- note removed: "1.8V"

Commit message: Almost Complete Schematic
Parts:
- R17, R18, R19, R20: value 10K -> 3.3K
Connections:
- net SDA: no longer IC2.4 (SDA), R18.2, U6.3 (SDAA)
- new net SDA_BAR: IC2.4 (SDA), R18.2, U6.3 (SDAA)
Other:
- note added: "Level Shifting"
Changed lines of the file:
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@@
 	(generator_version "10.0")
 	(paper "A4")
+	(rectangle
+		(start 49.53 63.5)
+		(end 125.73 133.35)
+		(stroke
+			(width 0)
+			(type dash)
+		)
+		(fill
+			(type none)
+		)
+	)
+	(text "Level Shifting"
+		(exclude_from_sim no)
+		(at 55.88 62.738 0)
+		(effects
+			(font
+				(size 1.27 1.27)
+			)
+		)
+	)
 	(junction
 		(at 72.39 80.01)
@@
 	(wire
 		(pts
-			(xy 121.92 107.95) (xy 128.27 107.95)
+			(xy 121.92 107.95) (xy 125.73 107.95)
 		)
 		(stroke
@@
 		)
 	)
-	(label "SDA"
-		(at 128.27 107.95 0)
+	(label "SDA_BAR"
+		(at 125.73 107.95 0)
 		(effects
 			(font
@@
 		)
 	)
-	(label "SDA"
+	(label "SDA_BAR"
 		(at 147.32 123.19 270)
 		(effects
@@
 			)
 		)
-		(property "Value" "10K"
+		(property "Value" "3.3K"
 			(at 76.2 96.52 90)
 			(show_name no)
@@
 			)
 		)
-		(property "Value" "10K"
+		(property "Value" "3.3K"
 			(at 118.11 96.52 90)
 			(show_name no)
@@
 			)
 		)
-		(property "Value" "10K"
+		(property "Value" "3.3K"
 			(at 67.31 96.52 90)
 			(show_name no)
@@
 			)
 		)
-		(property "Value" "10K"
+		(property "Value" "3.3K"
 			(at 109.22 96.52 90)
 			(show_name no)
