File: IST-8310.kicad_sch (KiCad schematic)
At the start: 8 parts, among them U5 IST8310

Commit message: progress
Parts:
- added C56: 100nF, Capacitor_SMD:C_0805_2012Metric, symbol Device:C
- added C57: 1uF, Capacitor_SMD:C_0805_2012Metric, symbol Device:C
- added FB5: 1K/0.1A, Inductor_SMD:L_0603_1608Metric, symbol Device:FerriteBead_Small
- added NT5: Tie_MAG_Rail, NetTie:NetTie-2_SMD_Pad0.5mm, symbol Device:NetTie_2
- C46: value 100nF -> 1uF
Connections:
- net GND: now also C56.1, C57.1
- net VDDMAG: now also C56.2, C57.2, FB5.2; no longer C45.2, C46.2, R21.1, R22.1, R23.1, U5.13 (DVDD), U5.7 (VPP)
- new net VDDMAG_IO: C45.2, C46.2, FB5.1, NT5.2, R21.1, R22.1, R23.1, U5.13 (DVDD), U5.7 (VPP)
- new net VDD_3V3_S: NT5.1
Other:
- moved on the sheet: C45, C46

Commit message: Almost Complete Schematic
Parts:
- R21, R22: value 10K -> 3.3K
Changed lines of the file:
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@@
 			)
 		)
-		(property "Value" "10K"
+		(property "Value" "3.3K"
 			(at 129.54 93.98 90)
 			(show_name no)
@@
 			)
 		)
-		(property "Value" "10K"
+		(property "Value" "3.3K"
 			(at 119.38 93.98 90)
 			(show_name no)
