File: SD_Card.kicad_sch (KiCad schematic)
At the start: 18 parts, among them IC4 EMIF06-HSD03F3, J1 Micro_SD_Card_Det_Hirose_DM3AT, Q1 FDN340P, Q2 BC847

Commit message: Almost Complete Schematic
Parts:
- added C75: 100nF, Capacitor_SMD:C_0805_2012Metric, symbol Device:C
- added R82: 47K, Resistor_SMD:R_0805_2012Metric, symbol Device:R
- R36: value 1K -> 470R
Connections:
- net GND: now also D1.1 (K), C75.1; no longer D1.2 (A)
- net SD_CK: now also R82.2
- net SD_DET: now also C75.2
- net VDD_SD: now also R82.1
- net at R36.2: now also D1.2 (A); no longer D1.1 (K)
Other:
- moved on the sheet: D1
