File: STM32L552QEIxQ.kicad_sch (KiCad schematic)
At the start: 30 parts, among them U1 STM32L552QEIxQ, U2 TL431DBZ, Y1 ABM8G-24.000MHZ-4Y-T

Commit message: asdad
Parts:
- added Y2: ABS06-32.768KHZ-1-T, ABS06, symbol ABS06:ABS06-32.768KHZ-1-T
Changed lines of the file:
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@@
+	)
+	(symbol
+		(lib_id "ABS06:ABS06-32.768KHZ-1-T")
+		(at 236.22 148.59 0)
+		(unit 1)
+		(body_style 1)
+		(exclude_from_sim no)
+		(in_bom yes)
+		(on_board yes)
+		(in_pos_files yes)
+		(dnp no)
+		(fields_autoplaced yes)
+		(property "Reference" "Y2"
+			(at 241.3 139.7 0)
+			(show_name no)
+			(do_not_autoplace no)
+			(effects
+				(font
+					(size 1.27 1.27)
+				)
+			)
+		)
+		(property "Value" "ABS06-32.768KHZ-1-T"
+			(at 241.3 142.24 0)
+			(show_name no)
+			(do_not_autoplace no)
+			(effects
+				(font
+					(size 1.27 1.27)
+				)
+			)
+		)
+		(property "Footprint" "ABS06"
+			(at 245.11 244.78 0)
+			(hide yes)
+			(show_name no)
+			(do_not_autoplace no)
+			(effects
+				(font
+					(size 1.27 1.27)
+				)
+				(justify left top)
+			)
+		)
+		(property "Datasheet" "https://abracon.com/Resonators/ABS06.pdf"
+			(at 245.11 344.78 0)
+			(hide yes)
+			(show_name no)
+			(do_not_autoplace no)
+			(effects
+				(font
+					(size 1.27 1.27)
+				)
+				(justify left top)
+			)
+		)
+		(property "Description" "32.768 kHz +/-10ppm Crystal 12.5pF 90 kOhms 2-SMD, No Lead"
+			(at 236.22 148.59 0)
+			(hide yes)
+			(show_name no)
+			(do_not_autoplace no)
+			(effects
+				(font
+					(size 1.27 1.27)
+				)
+			)
+		)
+		(property "Height" "0.6"
+			(at 245.11 544.78 0)
+			(hide yes)
+			(show_name no)
+			(do_not_autoplace no)
+			(effects
+				(font
+					(size 1.27 1.27)
+				)
+				(justify left top)
+			)
+		)
+		(property "Manufacturer_Name" "ABRACON"
+			(at 245.11 644.78 0)
+			(hide yes)
+			(show_name no)
+			(do_not_autoplace no)
+			(effects
+				(font
+					(size 1.27 1.27)
+				)
+				(justify left top)
+			)
+		)
+		(property "Manufacturer_Part_Number" "ABS06-32.768KHZ-1-T"
+			(at 245.11 744.78 0)
+			(hide yes)
+			(show_name no)
+			(do_not_autoplace no)
+			(effects
+				(font
+					(size 1.27 1.27)
+				)
+				(justify left top)
+			)
+		)
+		(property "Mouser Part Number" "815-ABS06-32.7K-1-T"
+			(at 245.11 844.78 0)
+			(hide yes)
+			(show_name no)
+			(do_not_autoplace no)
+			(effects
+				(font
+					(size 1.27 1.27)
+				)
+				(justify left top)
+			)
+		)
+		(property "Mouser Price/Stock" "https://www.mouser.co.uk/ProductDetail/ABRACON/ABS06-32.768KHZ-1-T?qs=3LVMET7lfiOVpH4K9yAPuw%3D%3D"
+			(at 245.11 944.78 0)
+			(hide yes)
+			(show_name no)
+			(do_not_autoplace no)
+			(effects
+				(font
+					(size 1.27 1.27)
+				)
+				(justify left top)
+			)
+		)
+		(property "Arrow Part Number" "ABS06-32.768KHZ-1-T"
+			(at 245.11 1044.78 0)
+			(hide yes)
+			(show_name no)
+			(do_not_autoplace no)
+			(effects
+				(font
+					(size 1.27 1.27)
+				)
+				(justify left top)
+			)
+		)
+		(property "Arrow Price/Stock" "https://www.arrow.com/en/products/abs06-32.768khz-1-t/abracon?utm_currency=USD&region=nac"
+			(at 245.11 1144.78 0)
+			(hide yes)
+			(show_name no)
+			(do_not_autoplace no)
+			(effects
+				(font
+					(size 1.27 1.27)
+				)
+				(justify left top)
+			)
+		)
+		(pin "1"
+		)
+		(pin "2"
+		)
+		(instances
+			(project "141 FC"
+				(path "/524bae94-30c3-4d47-8232-d1fa64637976/40473a26-0dec-4a83-80ba-cc1bd63742f6"
+					(reference "Y2")
+					(unit 1)
+				)
+			)
+		)
 	)
 	(symbol

Commit message: Commit_1
Parts:
- removed C1: 4.7uF, Capacitor_SMD:C_0805_2012Metric, symbol Device:C
- removed L1: 4.7uH, Inductor_SMD:L_0805_2012Metric_Pad1.05x1.20mm_HandSolder, symbol Device:L
- removed NT1: NetTie_2, NetTie:NetTie-2_SMD_Pad0.5mm, symbol Device:NetTie_2
- removed U1: STM32L552QEIxQ, Package_BGA:UFBGA-132_7x7mm_Layout12x12_P0.5mm, symbol MCU_ST_STM32L5:STM32L552QEIxQ
- added C18, C19: 27pF, Capacitor_SMD:C_0805_2012Metric, symbol Device:C
- added C20, C21: 15pF, Capacitor_SMD:C_0805_2012Metric, symbol Device:C
- added C22, C28: 1uF, Capacitor_SMD:C_0805_2012Metric, symbol Device:C
- added C23, C24, C25, C26, C27: 100nF, Capacitor_SMD:C_0805_2012Metric, symbol Device:C
- added C29, C30: 2.2uF, Capacitor_SMD:C_0805_2012Metric, symbol Device:C
- added JP1: PDR, Jumper:SolderJumper-3_P2.0mm_Open_TrianglePad1.0x1.5mm_NumberLabels, symbol Jumper:SolderJumper_3_Open
- added R6, R7: 220R, Resistor_SMD:R_0805_2012Metric, symbol Device:R
- added R8: 10K, Resistor_SMD:R_0805_2012Metric, symbol Device:R
- added U3: STM32H723ZGIx, Package_BGA:UFBGA-144_7x7mm_Layout12x12_P0.5mm, symbol MCU_ST_STM32H7:STM32H723ZGIx
- C12: value 10nF -> 100nF
- C9: value 4.7uF -> 100nF
- R4, R5: value 100K -> 10K
- Y2: footprint ABS06 -> ABS06:ABS06
Connections:
- net +Vref: now also U3.L1 (VREF+)
- net GND: now also R5.1, Y1.2 (GND_1), Y1.4 (GND_2), C18.2, C19.2, C20.2, C21.2, C22.1, C23.1, C24.1, C25.1, C26.1, C27.2, C28.1, C29.1, C30.1, JP1.3 (B), U3.D2 (VSS), U3.E6 (VSS), U3.E7 (VSS), U3.G10 (VSS), U3.G4 (VSS), U3.G8 (VSS), U3.H5 (VSS), U3.H6 (VSS), U3.J1 (VSSA), U3.K1 (VREF-); no longer S2.2
- net RST: now also U3.F1 (NRST); no longer R5.2, S2.1, S2.3
- net SWDCLK: now also U3.A11 (PA14(JTCK)
- net SWDIO: now also U3.A12 (PA13(JTMS)
- net SWO: now also U3.A7 (PB3(JTDO)
- net USB_DM: now also U3.C12 (PA11)
- net USB_DP: now also U3.B12 (PA12)
- net VDDA: now also U3.M1 (VDDA)
- net VDDMCU: now also S2.2, C24.2, C25.2, C26.2, JP1.1 (A), U3.D3 (VDD), U3.F10 (VDD), U3.F4 (VDD), U3.F5 (VDD), U3.F6 (VDD), U3.F7 (VDD), U3.F8 (VDD), U3.F9 (VDD), U3.G5 (VDD), U3.G6 (VDD), U3.G7 (VDD)
- net OSC32_IN: now reaches Y2.1
- net OSC32_IN: now also C20.1, U3.B1 (PC14)
- net OSC32_OUT: now reaches Y2.2
- net OSC32_OUT: now also C21.1, U3.C1 (PC15)
- net OSC_IN: now reaches Y1.1 (XTAL_1)
- net OSC_IN: now also C18.1, U3.D1 (PH0)
- net at Y1.3 (XTAL_2): now also C19.1, R7.1
- net at BT1.1 (+): now also C27.1, C28.2, U3.C2 (VBAT)
- new net: R6.2, U3.D5 (BOOT0)
- new net: R8.1, U3.E5 (PDR_ON)
- new net: C30.2, U3.G9 (VCAP)
- new net: C29.2, U3.H7 (VCAP)
- new net BOOT0: R5.2, R6.1, S2.1, S2.3
- new net IMU_1_MISO: U3.A6 (PB4(NJTRST))
- new net IMU_1_MOSI: U3.A9 (PD7)
- new net IMU_1_SCK: U3.C8 (PG11)
- new net OSC_OUT: R7.2, U3.E1 (PH1)
- new net OSPI_CLK: U3.G1 (PF10)
- new net OSPI_D0: U3.E11 (PC9)
- new net OSPI_D1: U3.B11 (PC10)
- new net OSPI_D2: U3.A3 (PE2)
- new net OSPI_D3: U3.F3 (PF6)
- new net OSPI_NCS: U3.B10 (PC11)
- new net PDR_ON: JP1.2 (C), R8.2
- new net VDDUSB: C22.2, C23.2, U3.C11 (VDD33USB)
Other:
- note added: "BOOT Selection"
- note added: "By-Pass Capacitors(VDDUSB)"
- note added: "HSE"
- note added: "LSE"
- note added: "Power Down Reset Setting"
- note removed: "BOOT"
- note removed: "By-Pass Capacitors(IO2)"
- moved on the sheet: BT1, C10, C17, C2, C3, C4, C5, C6, C7, C8, C9, R5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

Commit message: progress
Parts:
- removed C16, C17: 100nF, Capacitor_SMD:C_0805_2012Metric, symbol Device:C
- added FB1: 1K/0.1A, Inductor_SMD:L_0603_1608Metric, symbol Device:FerriteBead_Small
- added NT1: Tie_MCU_Rail, NetTie:NetTie-2_SMD_Pad0.5mm, symbol Device:NetTie_2
- R1: value 220R -> 1K
Connections:
- net VDDUSB is gone; now on net VDDMCU: C22.2, C23.2, U3.C11 (VDD33USB)
- net GND: now also S1.MP1, S1.MP2, S2.MP1, S2.MP2
- net VDDA: now also FB1.2
- net VDDMCU: now also FB1.1, NT1.2
- new net VDD: NT1.1
Other:
- note added: "1-2 Default"
- note added: "Power Tree"

Commit message: Almost Complete Schematic
Parts:
- added D5: LED, LED_SMD:LED_0805_2012Metric, symbol Device:LED
- added D6, D7, D8: PESD3V3X1BL,315, PESD3V3X1BL:PESD5V0S1BL315, symbol PESD3V3X1BL_315:PESD3V3X1BL,315
- added J10: SWDIO, Connector_Wire:SolderWirePad_1x01_SMD_1x2mm, symbol Connector:Conn_01x01_Pin
- added J11: SWCLK, Connector_Wire:SolderWirePad_1x01_SMD_1x2mm, symbol Connector:Conn_01x01_Pin
- added J12: SWO, Connector_Wire:SolderWirePad_1x01_SMD_1x2mm, symbol Connector:Conn_01x01_Pin
- added J13: VCC, Connector_Wire:SolderWirePad_1x01_SMD_1x2mm, symbol Connector:Conn_01x01_Pin
- added J14: GND, Connector_Wire:SolderWirePad_1x01_SMD_1x2mm, symbol Connector:Conn_01x01_Pin
- added R54: 470R, Resistor_SMD:R_0805_2012Metric, symbol Device:R
- added R71: 0R, Resistor_SMD:R_0805_2012Metric, symbol Device:R
Connections:
- net GND: now also D5.1 (K), D6.2 (K2), D7.2 (K2), D8.2 (K2), J14.1 (Pin_1)
- net IMU_1_MISO: now also U3.L3 (PA6); no longer U3.A6 (PB4(NJTRST))
- net IMU_1_MOSI: now also U3.M3 (PA7); no longer U3.A9 (PD7)
- net IMU_1_SCK: now also U3.K3 (PA5); no longer U3.C8 (PG11)
- net OSPI_D0: now also U3.G3 (PF8); no longer U3.E11 (PC9)
- net OSPI_D1: now also U3.G2 (PF9); no longer U3.B11 (PC10)
- net OSPI_D2: now also U3.F2 (PF7); no longer U3.A3 (PE2)
- net OSPI_NCS: now also U3.H11 (PG6); no longer U3.B10 (PC11)
- net SWDCLK: now also D7.1 (K1), J11.1 (Pin_1)
- net SWDIO: now also D6.1 (K1), J10.1 (Pin_1)
- net SWO: now also D8.1 (K1), J12.1 (Pin_1)
- net VDDMCU: now also R71.2
- net BLE_RTS: now reaches U3.A10 (PA15(JTDI))
- net SBUS_2: now reaches U3.A2 (PE3)
- net T1: now reaches U3.A4 (PE1)
- net R1: now reaches U3.A5 (PE0)
- net RX_RADIO: now reaches U3.A8 (PD6)
- net I2S FS: now reaches U3.B2 (PE4)
- net I2S SCK: now reaches U3.B3 (PE5)
- net CAN_SLEEP: now reaches U3.B4 (PE6)
- net CAN_TX: now reaches U3.B5 (PB9)
- net SERVO 1: now reaches U3.B8 (PG12)
- net TX_RADIO: now reaches U3.B9 (PD5)
- net SD_CLK: now reaches U3.C10 (PC12)
- net BAR_SDA: now reaches U3.C3 (PF0)
- net BAR_SCL: now reaches U3.C4 (PF1)
- net CAN_RX: now reaches U3.C5 (PB8)
- net MAG_SCL: now reaches U3.C6 (PB6)
- net MAG_RST: now reaches U3.C7 (PG14)
- net BLE_TX: now reaches U3.D10 (PD1)
- net BLE_RST: now reaches U3.D11 (PA10)
- net VBUS_SENSE: now reaches U3.D12 (PA9)
- net SERVO 2: now reaches U3.D4 (PF2)
- net MAG_SDA: now reaches U3.D6 (PB7)
- net MAG_INT: now reaches U3.D7 (PG13)
- net BLE_POWER: now reaches U3.D9 (PD3)
- net BLE_RX: now reaches U3.E10 (PD0)
- net SD_PWR: now reaches U3.E12 (PA8)
- net SERVO 3: now reaches U3.E2 (PF3)
- net SD_CMD: now reaches U3.E9 (PD2)
- net SD_D0: now reaches U3.F11 (PC8)
- net R4: now reaches U3.F12 (PC7)
- net FLASH_RST: now reaches U3.G11 (PG8)
- net T4: now reaches U3.G12 (PC6)
- net SD_DET: now reaches U3.H12 (PG5)
- net I2S_SD: now reaches U3.H2 (PC1)
- net M2: now reaches U3.H8 (PE11)
- net IMU_1_nCS_G: now reaches U3.J2 (PA0)
- net IMU_1_nCS_A: now reaches U3.J3 (PA4)
- net IMU_1_INT: now reaches U3.J4 (PC4)
- net SDA: now reaches U3.K10 (PD13)
- net R2: now reaches U3.K11 (PD14)
- net T2: now reaches U3.K12 (PD15)
- net NEO PIXEL 3: now reaches U3.K5 (PF13)
- net M1: now reaches U3.K7 (PE9)
- net M3: now reaches U3.K8 (PE13)
- net R3: now reaches U3.K9 (PD9)
- net SCL: now reaches U3.L10 (PD12)
- net IMU_2_MISO: now reaches U3.L11 (PB14)
- net IMU_2_MOSI: now reaches U3.L12 (PB15)
- net BLE_CTS: now reaches U3.L4 (PB0)
- net NEO PIXEL 2: now reaches U3.L5 (PF12)
- net M4: now reaches U3.L8 (PE14)
- net T3: now reaches U3.L9 (PD8)
- net IMU_2_INT_2: now reaches U3.M10 (PB11)
- net IMU_2_nCS: now reaches U3.M11 (PB12)
- net IMU_2_SCK: now reaches U3.M12 (PB13)
- net NEO PIXEL 1: now reaches U3.M5 (PF11)
- net NEO PIXEL 4: now reaches U3.M6 (PF14)
- net IMU_2_INT_1: now reaches U3.M9 (PB10)
- net +5V: now reaches R1.1
- new net: J13.1 (Pin_1), R71.1
- new net: D5.2 (A), R54.1
- new net I2S MCK: U3.A3 (PE2)
- new net SBUS_1: U3.A6 (PB4(NJTRST))
- new net SD_D1: U3.E11 (PC9)
- new net SD_D2: U3.B11 (PC10)
- new net SD_D3: U3.B10 (PC11)
- new net USER_LED: R54.2
Other:
- note added: "DEBUG"
